File: RawWaves_1-0a.brd (EAGLE design)
At the start: 107 x 20 mm, 53 parts, among them IC1 LM1117MP-5.0, IC4 TL074, U1 TEENSY_3.1_TW, X1 VERT_SD_CARD_REV2

Commit message: Add Voltage Supervisor
Parts:
- added POGO: (no value), wirepad:1,6/0,8
- added R22: 100k, rcl:R0805
- added U2: MIC803-26D4VM3TR, Micrel_By_element14_Batch_1:SOT95P232X110-3N
- moved D6 41.2 mm to (44.5, 4.21), turned to 180 degrees
- moved D9 39.8 mm to (92.7, 17.9), turned to 0 degrees
- moved D5 34.9 mm to (92.3, 9.44), turned to 0 degrees
- moved R19 33.9 mm to (40.0, 2.16), turned to 90 degrees
- moved R1 22.3 mm to (81.9, 14.1), turned to 270 degrees
- moved F1 17.2 mm to (29.6, 12.8), turned to 90 degrees
- moved C1 14.3 mm to (52.7, 10.9)
- moved R4 14.2 mm to (52.7, 13.0)
- moved R3 11.9 mm to (51.7, 16.0), turned to 90 degrees
- moved D2 11.1 mm to (28.4, 16.9), turned to 180 degrees
- moved C5 10.3 mm to (70.3, 8.49)
- moved C10 9.94 mm to (20.4, 12.3)
- moved R12 9.27 mm to (101.9, 5.71), turned to 0 degrees
- moved R18 8.69 mm to (4.50, 8.58)
- moved R5 8.02 mm to (64.0, 7.75)
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Connections:
- new net N$17: POGO.1, R22.1, U2.2
- net +3.3V: now also R22.2, U2.3
- net DGND: now also U2.1
Routing:
- net GND: track 219.6 -> 271.2 mm, vias 2 -> 1
- net +3.3V: track 133.7 -> 87.5 mm
- net DGND: track 75.0 -> 45.6 mm, vias 3 -> 1
- net N$1: track 36.7 -> 10.2 mm
- net +12V_INLET: track 28.3 -> 9.13 mm
- net N$5: track 19.5 -> 32.9 mm
- net AUDIO_OUT: track 90.1 -> 77.7 mm
- net -12V_INLET: track 20.4 -> 8.05 mm
- net PIN22/A8: track 34.0 -> 22.1 mm, vias 0 -> 1
- net LED2: track 37.6 -> 27.1 mm, vias 1 -> 0
- net CHANNEL_CV: track 72.0 -> 63.0 mm, vias 4 -> 2
- net -12V: track 61.9 -> 70.5 mm, vias 4 -> 2
- net N$8: track 12.2 -> 3.61 mm
- net LED4: track 37.6 -> 30.7 mm, vias 1 -> 0
- net N$17: track 0.00 -> 6.72 mm
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Other:
- board text added: "Raw Waves v1.0 by Sherpa Modular, licensed under CC-BY-SA 3.0 This is a derivative work from "Radio Music" by Tom Whitwell, Which has been used under CC-BY-SA 3.0 www.sherpamodular.com"
- board text added: "You're a curious one. I like you."
- board text added: "■"
- board text removed: "Raw Waves v1.0, by Sherpa Modular www.sherpamodular.com licensed under CC-BY-SA 3.0 This is a derivative work from "Radio Music" by Music Thing Modular. Used under CC-BY-SA 3.0"
