File: RawWaves_v1-1.sch (EAGLE design)
At the start: 56 parts, among them IC1 LM1117MP-5.0, IC4 TL074, U1 TEENSY_3.1_TW, U2 MIC803-26D4VM3TR, X1 VERT_SD_CARD_REV2

Commit message: Widen Pogo Hole
Replaced "Pogo 1.6/0.8" with "Pogo 1.6/0.9"
Parts:
- removed POGO: (no value), wirepad:1,6/0,8
- added PAD1: (no value), wirepad:1,6/0,9
Connections:
- net N$17: now also PAD1.P; no longer POGO.P
Changed lines of the file:
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@@
 <part name="F1" library="polyfuse-smd_10" deviceset="?" device="1206L" technology="020"/>
 <part name="IC1" library="lm1117" deviceset="LM1117?-*" device="MP" technology="5.0"/>
-<part name="POGO" library="wirepad" library_urn="urn:adsk.eagle:library:412" deviceset="1,6/0,8" device="" package3d_urn="urn:adsk.eagle:package:30830/1"/>
 <part name="U2" library="Micrel_By_element14_Batch_1" deviceset="MIC803-26D4VM3TR" device=""/>
 <part name="R22" library="rcl" library_urn="urn:adsk.eagle:library:334" deviceset="R-US_" device="R0805" package3d_urn="urn:adsk.eagle:package:23553/2" value="100k"/>
+<part name="PAD1" library="wirepad" library_urn="urn:adsk.eagle:library:412" deviceset="1,6/0,9" device="" package3d_urn="urn:adsk.eagle:package:30840/1"/>
 </parts>
 <sheets>
@@
 <attribute name="VALUE" x="287.02" y="12.7" size="1.778" layer="96"/>
 </instance>
-<instance part="POGO" gate="P" x="96.52" y="-71.12" smashed="yes" rot="R180">
-<attribute name="NAME" x="97.663" y="-72.9742" size="1.778" layer="95" rot="R180"/>
-<attribute name="VALUE" x="97.663" y="-67.818" size="1.778" layer="96" rot="R180"/>
-</instance>
 <instance part="U2" gate="A" x="50.8" y="-71.12" smashed="yes">
 <attribute name="NAME" x="62.5348" y="-63.881" size="2.0828" layer="95" ratio="10" rot="SR0"/>
@@
 <attribute name="NAME" x="74.93" y="-62.4586" size="1.778" layer="95" rot="R180"/>
 <attribute name="VALUE" x="74.93" y="-57.658" size="1.778" layer="96" rot="R180"/>
+</instance>
+<instance part="PAD1" gate="1" x="96.52" y="-71.12" smashed="yes" rot="R180">
+<attribute name="NAME" x="97.663" y="-72.9742" size="1.778" layer="95" rot="R180"/>
+<attribute name="VALUE" x="97.663" y="-67.818" size="1.778" layer="96" rot="R180"/>
 </instance>
 </instances>
@@
 <segment>
 <pinref part="U2" gate="A" pin="~RESET"/>
-<pinref part="POGO" gate="P" pin="P"/>
 <wire x1="93.98" y1="-71.12" x2="86.36" y2="-71.12" width="0.1524" layer="91"/>
 <pinref part="R22" gate="G$1" pin="1"/>
@@
 <wire x1="86.36" y1="-60.96" x2="86.36" y2="-71.12" width="0.1524" layer="91"/>
 <junction x="86.36" y="-71.12"/>
-</segment>
-</net>
+<pinref part="PAD1" gate="1" pin="P"/>
+</segment>
+</net>
